File: electronics/main-v2/main.kicad_pcb (KiCad board)
At the start: 2 copper layers, 82 x 52 mm, 19 parts, among them J1 Port, SW1 SW_Push, SW2 SW_Push, SW3 SW_Push, U1 ATmega88V-10PU, U2 DS18B20, U3 BU9796AMUV-E2

Commit message: boards
Other:
- board text added: "CALIBRATE ME!"
Changed lines of the file:
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@@
   (general
     (thickness 1.6)
-    (drawings 26)
+    (drawings 63)
     (tracks 212)
     (zones 0)
@@
   (page A4)
   (layers
-    (0 F.Cu signal hide)
-    (31 B.Cu signal hide)
-    (32 B.Adhes user)
-    (33 F.Adhes user)
-    (34 B.Paste user)
+    (0 F.Cu signal)
+    (31 B.Cu signal)
+    (32 B.Adhes user hide)
+    (33 F.Adhes user hide)
+    (34 B.Paste user hide)
     (35 F.Paste user hide)
     (36 B.SilkS user)
     (37 F.SilkS user)
-    (38 B.Mask user)
+    (38 B.Mask user hide)
     (39 F.Mask user hide)
     (40 Dwgs.User user)
@@
       (layerselection 0x010fc_ffffffff)
       (usegerberextensions false)
-      (usegerberattributes true)
-      (usegerberadvancedattributes true)
+      (usegerberattributes false)
+      (usegerberadvancedattributes false)
       (creategerberjobfile true)
       (excludeedgelayer true)
@@
       (outputformat 1)
       (mirror false)
-      (drillshape 1)
+      (drillshape 0)
       (scaleselection 1)
-      (outputdirectory ""))
+      (outputdirectory "../main-v2-pcbway/"))
   )
   (net 0 "")
@@
     (add_net "Net-(R4-Pad2)")
     (add_net "Net-(R5-Pad2)")
-    (add_net "Net-(U1-Pad11)")
-    (add_net "Net-(U1-Pad12)")
-    (add_net "Net-(U1-Pad13)")
-    (add_net "Net-(U1-Pad14)")
-    (add_net "Net-(U1-Pad16)")
-    (add_net "Net-(U1-Pad20)")
-    (add_net "Net-(U1-Pad21)")
-    (add_net "Net-(U1-Pad22)")
-    (add_net "Net-(U1-Pad24)")
-    (add_net "Net-(U1-Pad3)")
-    (add_net "Net-(U1-Pad4)")
-    (add_net "Net-(U1-Pad5)")
-    (add_net "Net-(U1-Pad6)")
-    (add_net "Net-(U3-Pad25)")
     (add_net PIN-BTN-MINUS)
     (add_net PIN-BTN-MODE)
@@
     )
     (fp_text value BU9796AMUV-E2 (at 0 -3.32) (layer B.Fab)
-      (effects (font (size 1 1) (thickness 0.15)) (justify mirror))
-    )
-    (fp_text user %R (at 0 0) (layer B.Fab)
       (effects (font (size 1 1) (thickness 0.15)) (justify mirror))
     )
@@
     (fp_line (start 2.62 -2.62) (end 2.62 2.62) (layer B.CrtYd) (width 0.05))
     (fp_line (start 2.62 2.62) (end -2.62 2.62) (layer B.CrtYd) (width 0.05))
+    (fp_text user %R (at 0 0) (layer B.Fab)
+      (effects (font (size 1 1) (thickness 0.15)) (justify mirror))
+    )
     (pad "" smd roundrect (at 0.82 -0.82 180) (size 0.66 0.66) (layers B.Paste) (roundrect_rratio 0.25))
     (pad "" smd roundrect (at 0.82 0 180) (size 0.66 0.66) (layers B.Paste) (roundrect_rratio 0.25))
@@
       (effects (font (size 1 1) (thickness 0.15)))
     )
-    (fp_text user %R (at 5.08 0 90) (layer F.Fab)
-      (effects (font (size 1 1) (thickness 0.15)))
-    )
     (fp_line (start 1.93 -1.25) (end 1.93 1.25) (layer F.Fab) (width 0.1))
     (fp_line (start 1.93 1.25) (end 8.23 1.25) (layer F.Fab) (width 0.1))
@@
     (fp_line (start 11.21 1.5) (end 11.21 -1.5) (layer F.CrtYd) (width 0.05))
     (fp_line (start 11.21 -1.5) (end -1.05 -1.5) (layer F.CrtYd) (width 0.05))
+    (fp_text user %R (at 5.08 0 90) (layer F.Fab)
+      (effects (font (size 1 1) (thickness 0.15)))
+    )
     (pad 2 thru_hole oval (at 10.16 0 90) (size 1.6 1.6) (drill 0.8) (layers *.Cu *.Mask)
       (net 34 "Net-(R5-Pad2)"))
@@
     )
     (fp_text value 10k (at 5.08 2.37 90) (layer F.Fab)
-      (effects (font (size 1 1) (thickness 0.15)))
-    )
-    (fp_text user %R (at 5.08 0 90) (layer F.Fab)
       (effects (font (size 1 1) (thickness 0.15)))
     )
@@
     (fp_line (start 11.21 1.5) (end 11.21 -1.5) (layer F.CrtYd) (width 0.05))
     (fp_line (start 11.21 -1.5) (end -1.05 -1.5) (layer F.CrtYd) (width 0.05))
+    (fp_text user %R (at 5.08 0 90) (layer F.Fab)
+      (effects (font (size 1 1) (thickness 0.15)))
+    )
     (pad 2 thru_hole oval (at 10.16 0 90) (size 1.6 1.6) (drill 0.8) (layers *.Cu *.Mask)
       (net 33 "Net-(R4-Pad2)"))
@@
       (effects (font (size 1 1) (thickness 0.15)) (justify mirror))
     )
-    (fp_text user %R (at 0 0) (layer B.Fab)
-      (effects (font (size 0.4 0.4) (thickness 0.06)) (justify mirror))
-    )
     (fp_line (start -0.8 -0.4) (end -0.8 0.4) (layer B.Fab) (width 0.1))
     (fp_line (start -0.8 0.4) (end 0.8 0.4) (layer B.Fab) (width 0.1))
@@
     (fp_line (start 1.48 0.73) (end 1.48 -0.73) (layer B.CrtYd) (width 0.05))
     (fp_line (start 1.48 -0.73) (end -1.48 -0.73) (layer B.CrtYd) (width 0.05))
+    (fp_text user %R (at 0 0) (layer B.Fab)
+      (effects (font (size 0.4 0.4) (thickness 0.06)) (justify mirror))
+    )
     (pad 2 smd roundrect (at 0.775 0) (size 0.9 0.95) (layers B.Cu B.Paste B.Mask) (roundrect_rratio 0.25)
       (net 1 GND))
@@
   (gr_line (start 112 88) (end 118.5 88) (layer Edge.Cuts) (width 0.05))
   (gr_line (start 112 91) (end 112 88) (layer Edge.Cuts) (width 0.05))
-  (gr_text "RST\n\nSCK\n\nMISO\n\nMOSI\n\nVCC\n\nGND\n" (at 148.336 86.106 90) (layer F.SilkS)
+  (gr_text "RST\n\nSCK\n\nMISO\n\nMOSI\n\nVCC\n\nGND\n" (at 148.25 86 90) (layer F.SilkS)
     (effects (font (size 0.75 0.75) (thickness 0.15)) (justify left))
   )
@@
   (gr_line (start 161 47) (end 161 83) (layer Edge.Cuts) (width 0.05))
   (gr_line (start 82 39) (end 158 39) (layer Edge.Cuts) (width 0.05))
+  (gr_text "CALIBRATE ME!" (at 128.75 68.25 90) (layer F.SilkS)
+    (effects (font (size 1.32 1.32) (thickness 0.17)))
+  )
+  (gr_line (start 114.6 67.375) (end 114.4 67.7) (layer F.SilkS) (width 0.4))
+  (gr_line (start 126.691057 61.199003) (end 126.691057 75.449003) (layer F.SilkS) (width 0.4))
+  (gr_line (start 121.446622 61.278843) (end 121.55 62) (layer F.SilkS) (width 0.4))
+  (gr_line (start 122.468619 62.105105) (end 122.25 63.2) (layer F.SilkS) (width 0.4))
+  (gr_line (start 120.44899 62.105105) (end 120.75 63.2) (layer F.SilkS) (width 0.4))
+  (gr_line (start 121.463629 64.116522) (end 121.468474 67.5) (layer F.SilkS) (width 0.4))
+  (gr_line (start 123.45 67.6) (end 119.479506 67.597569) (layer F.SilkS) (width 0.4))
+  (gr_line (start 123.15 66.604539) (end 119.722184 66.606243) (layer F.SilkS) (width 0.4))
+  (gr_line (start 122.990423 64.209165) (end 122.989451 65.721059) (layer F.SilkS) (width 0.4))
+  (gr_line (start 119.950972 64.188106) (end 119.95 65.7) (layer F.SilkS) (width 0.4))
+  (gr_line (start 122.954333 65.782059) (end 119.959774 65.783763) (layer F.SilkS) (width 0.4))
+  (gr_line (start 122.95 64.901799) (end 119.955441 64.903503) (layer F.SilkS) (width 0.4))
+  (gr_line (start 122.95 64.1) (end 119.955441 64.101704) (layer F.SilkS) (width 0.4))
+  (gr_line (start 123.35 63.286029) (end 119.645427 63.286029) (layer F.SilkS) (width 0.4))
+  (gr_line (start 123.05 62.028728) (end 119.828904 62.028728) (layer F.SilkS) (width 0.4))
+  (gr_line (start 119.138444 62.415082) (end 118.25 61.7) (layer F.SilkS) (width 0.4))
+  (gr_line (start 118.25 61.3) (end 117.768474 62.1) (layer F.SilkS) (width 0.4))
+  (gr_line (start 117.75 62.1) (end 116.95 63.1) (layer F.SilkS) (width 0.4))
+  (gr_line (start 118.957705 65.367609) (end 118.957705 66.4) (layer F.SilkS) (width 0.4))
+  (gr_line (start 117.35 65.367609) (end 117.35 66.4) (layer F.SilkS) (width 0.4))
+  (gr_line (start 119.05 64.573204) (end 117.109082 64.573204) (layer F.SilkS) (width 0.4))
+  (gr_line (start 118.95 63.358675) (end 117.44188 63.358675) (layer F.SilkS) (width 0.4))
+  (gr_line (start 119.05 67.1) (end 117.108923 67.415935) (layer F.SilkS) (width 0.4))
+  (gr_line (start 118.145155 63.420387) (end 118.15 67.2) (layer F.SilkS) (width 0.4))
+  (gr_line (start 114.35 67.706549) (end 113.45 67.7) (layer F.SilkS) (width 0.4))
+  (gr_line (start 112.85 66.8) (end 112.15 66) (layer F.SilkS) (width 0.4))
+  (gr_line (start 114.610459 63.843865) (end 114.592265 67.4) (layer F.SilkS) (width 0.4))
+  (gr_line (start 113.668194 61.393021) (end 113.65 63.7) (layer F.SilkS) (width 0.4))
+  (gr_line (start 115.624816 65.207882) (end 111.746405 65.207882) (layer F.SilkS) (width 0.4))
+  (gr_line (start 115.65 63.77154) (end 111.771589 63.77154) (layer F.SilkS) (width 0.4))
+  (gr_line (start 115.25 62.371961) (end 112.076618 62.371961) (layer F.SilkS) (width 0.4))
+  (gr_line (start 109.65 64.2) (end 110.95 64.2) (layer F.SilkS) (width 0.4))
+  (gr_line (start 109.55 62) (end 109.55 66.7) (layer F.SilkS) (width 0.4))
+  (gr_line (start 111.05 62) (end 109.55 62) (layer F.SilkS) (width 0.4))
+  (gr_line (start 111.05 66.7) (end 111.05 62) (layer F.SilkS) (width 0.4))
+  (gr_line (start 109.55 66.7) (end 111.05 66.7) (layer F.SilkS) (width 0.4))
   (segment (start 148.59 57.404) (end 147.955 56.769) (width 0.2) (layer B.Cu) (net 1))
   (segment (start 151.13 57.404) (end 148.59 57.404) (width 0.2) (layer B.Cu) (net 1))
